File: KiCAD/Main Hub/MainBoard/MainBoard.kicad_pcb (KiCad board)
At the start: 2 copper layers, 100 x 100 mm, 119 parts, among them J1 Conn_01x08_Pin, J10 Conn_01x04_Pin, J11 Conn_01x04_Pin, J12 Conn_01x04_Pin, J13 Conn_01x04_Pin, J14 Conn_01x04_Pin, J15 Conn_01x04_Pin, J16 Conn_01x04_Pin, J17 Conn_01x04_Pin, J18 Conn_01x04_Pin, J19 Conn_01x04_Pin, J2 Conn_01x08_Pin, J20 Conn_01x08_Pin, J21 Conn_01x08_Pin, J3 Conn_02x06_Odd_Even, J4 Screw_Terminal_01x02, J5 Conn_01x08_Pin, J6 Conn_01x08_Pin, J7 Conn_01x08_Pin, J8 Conn_02x10_Odd_Even, J9 Conn_02x10_Odd_Even, U1 TCMT4100, U10 MCP23017_SS, U2 TCMT4100, U3 TCMT4100, U4 TCMT4100, U5 MCP23017_SS, U6 TCMT4100, U7 TCMT4100, U8 TCMT4100, U9 TCMT4100

Commit message: inital commit v1.1
Parts:
- moved PS1 218.2 mm to (-91.6, 31.5), turned to 0 degrees
- moved R33 215.3 mm to (-79.6, 96.7), turned to 0 degrees
- moved J4 195.6 mm to (-60.9, 52.7), turned to 0 degrees
- moved C1 191.9 mm to (-55.6, 70.0)
- moved C2 190.7 mm to (-55.6, 73.0)
- moved J15 176.4 mm to (-47.1, 100.3)
- moved J16 176.4 mm to (-47.1, 106.2)
- moved J17 176.4 mm to (-47.1, 112.0)
- moved J18 176.4 mm to (-47.1, 117.9)
- moved J19 176.4 mm to (-47.1, 123.8)
- moved A0 165.1 mm to (-56.7, 93.9)
- moved A1 165.0 mm to (-56.7, 97.7)
- moved A2 164.9 mm to (-56.7, 101.6)
- moved J10 160.4 mm to (-47.1, 71.1)
- moved J11 160.4 mm to (-47.1, 77.0)
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Routing:
- net GND2: track 239.1 -> 0.00 mm, vias 33 -> 0
- net SCK: track 187.5 -> 0.00 mm, vias 4 -> 0
- net SDA: track 173.7 -> 0.00 mm
- net INT: track 129.8 -> 0.00 mm, vias 3 -> 0
- net +5V: track 91.3 -> 0.00 mm, vias 49 -> 0
- net GND: track 48.6 -> 0.00 mm, vias 10 -> 0
- net Net-(U5-GPA0): track 33.4 -> 0.00 mm
- net +24V: track 30.7 -> 0.00 mm, vias 1 -> 0
- net Net-(U5-GPA1): track 30.6 -> 0.00 mm
- net Net-(U10-GPB7): track 29.3 -> 0.00 mm
- net Net-(U5-GPA2): track 27.5 -> 0.00 mm
- net Net-(U10-GPB6): track 27.5 -> 0.00 mm
- net Net-(U10-GPA0): track 24.9 -> 0.00 mm
- net Net-(U5-GPA3): track 24.8 -> 0.00 mm
- net Net-(U10-GPB5): track 24.8 -> 0.00 mm
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- removed copper zone on B.Cu, net +24V
- removed copper zone on B.Cu, net +5V
- removed copper zone on F.Cu, net GND
- removed copper zone on F.Cu, net GND2
Other:
- board outline removed
- board text removed: "24V"
- board text removed: "GND24|INT|SCK|SDA|5V|GND"
- board text removed: "Output"
- board text removed: "SCK|SDA|5V|GND"

Commit message: PSU pcb
Parts:
- removed the A0 at (-56.7, 93.9)
- removed the A1 at (-56.7, 97.7)
- removed the A2 at (-56.7, 101.6)
- removed A3: 5V-GND, Jumper:SolderJumper-3_P1.3mm_Open_Pad1.0x1.5mm
- removed A4, A5: Conn_01x03_Pin, Jumper:SolderJumper-3_P1.3mm_Open_Pad1.0x1.5mm
- removed the C1 at (-55.6, 70.0)
- removed the C2 at (-55.6, 73.0)
- removed C3: C, Capacitor_THT:CP_Radial_D6.3mm_P2.50mm
- removed C4, C6: C, Capacitor_SMD:C_0805_2012Metric_Pad1.18x1.45mm_HandSolder
- removed the C5 at (-6.15, 21.1)
- removed the H1 at (70.0, 53.1)
- removed the H2 at (147.0, 53.1)
- removed the H3 at (53.0, 91.4)
- removed the H4 at (147.0, 91.4)
- removed the H5 at (-24.2, 46.8)
- removed the H6 at (-24.2, 53.9)
- removed the J1 at (121.2, 97.6)
- removed the J10 at (-47.1, 71.1)
- removed the J11 at (-47.1, 77.0)
- removed the J12 at (-47.1, 82.8)
- removed the J13 at (-47.1, 88.7)
- removed the J14 at (-47.1, 94.5)
- removed the J15 at (-47.1, 100.3)
- removed the J16 at (-47.1, 106.2)
- removed the J17 at (-47.1, 112.0)
- removed the J18 at (-47.1, 117.9)
- removed J19: Conn_01x04_Pin, Connector_JST:JST_EH_B4B-EH-A_1x04_P2.50mm_Vertical
- removed the J2 at (146.0, 97.6)
- removed J20, J21, J5, J6, J7: Conn_01x08_Pin, Connector_JST:JST_EH_B8B-EH-A_1x08_P2.50mm_Vertical
- removed the J3 at (-33.8, 98.3)
- removed J4: Screw_Terminal_01x02, TerminalBlock_Phoenix:TerminalBlock_Phoenix_MKDS-1,5-2-5.08_1x02_P5.08mm_Horizontal
- removed the J8 at (83.2, 75.7)
- removed the J9 at (55.3, 75.7)
- removed PS1: IRM-10-24, Converter_ACDC:Converter_ACDC_MeanWell_IRM-10-xx_THT
- removed the R1 at (103.9, 90.2)
- removed the R10 at (127.3, 90.2)
- removed the R11 at (129.9, 90.2)
- removed the R12 at (132.5, 90.2)
- removed the R13 at (135.1, 90.2)
- removed the R14 at (137.7, 90.2)
- removed the R15 at (140.3, 90.2)
- removed the R16 at (142.9, 90.2)
- removed the R17 at (105.3, 76.3)
- removed the R18 at (108.2, 76.3)
- removed the R19 at (111.0, 76.3)
- removed the R2 at (106.5, 90.2)
- removed the R20 at (113.9, 76.3)
- removed the R21 at (116.7, 76.3)
- removed the R22 at (119.5, 76.3)
- removed the R23 at (122.4, 76.3)
- removed the R24 at (125.2, 76.3)
- removed the R25 at (128.1, 76.3)
- removed the R26 at (130.9, 76.3)
- removed the R27 at (133.8, 76.3)
- removed the R28 at (136.6, 76.3)
- removed the R29 at (139.5, 76.3)
- removed the R3 at (109.1, 90.2)
- removed the R30 at (142.3, 76.3)
- removed the R31 at (145.2, 76.3)
- removed the R32 at (148.0, 76.3)
- removed the R33 at (-79.6, 96.7)
- removed the R34 at (-26.5, 97.5)
- removed the R35 at (-26.5, 100.4)
- removed the R36 at (-26.5, 103.3)
- removed R37, R38, R39, R40, R41, R42, R43, R44, R45, R46, R47, R48, R49, R50, R51, R52, R53, R54, R55, R56, R57, R58, R59, R60, R61, R62, R63, R64, R65, R66, R67, R68, R69: R, Resistor_SMD:R_0805_2012Metric_Pad1.20x1.40mm_HandSolder
- removed the R4 at (111.7, 90.2)
- removed the R5 at (114.3, 90.2)
- removed the R6 at (116.9, 90.2)
- removed the R7 at (119.5, 90.2)
- removed the R8 at (122.1, 90.2)
- removed the R9 at (124.7, 90.2)
- removed the U1 at (109.9, 82.9)
- removed U10: MCP23017_SS, Package_SO:SSOP-28_5.3x10.2mm_P0.65mm
- removed the U2 at (121.2, 82.9)
- removed the U3 at (132.7, 82.8)
- removed the U4 at (144.1, 82.8)
- removed the U5 at (130.8, 62.5)
- removed U6, U7, U8, U9: TCMT4100, Package_SO:SOP-16_4.4x10.4mm_P1.27mm
- added A0: 5V-GND, Jumper:SolderJumper-3_P1.3mm_Open_Pad1.0x1.5mm, F.Cu at (126.0, 51.6)
- added A0: 5V-GND, Jumper:SolderJumper-3_P1.3mm_Open_Pad1.0x1.5mm, F.Cu at (126.0, 101.6)
- added A1: Conn_01x03_Pin, Jumper:SolderJumper-3_P1.3mm_Open_Pad1.0x1.5mm, F.Cu at (126.0, 54.5)
- added A1: Conn_01x03_Pin, Jumper:SolderJumper-3_P1.3mm_Open_Pad1.0x1.5mm, F.Cu at (126.0, 104.5)
- added A2: Conn_01x03_Pin, Jumper:SolderJumper-3_P1.3mm_Open_Pad1.0x1.5mm, F.Cu at (126.0, 107.4)
- added A2: Conn_01x03_Pin, Jumper:SolderJumper-3_P1.3mm_Open_Pad1.0x1.5mm, F.Cu at (126.0, 57.4)
- added C1: C, Capacitor_SMD:C_0805_2012Metric_Pad1.18x1.45mm_HandSolder, F.Cu at (147.4, 57.8)
- added C1: C, Capacitor_SMD:C_0805_2012Metric_Pad1.18x1.45mm_HandSolder, F.Cu at (147.4, 107.8)
- added C2: C, Capacitor_SMD:C_0805_2012Metric_Pad1.18x1.45mm_HandSolder, F.Cu at (147.4, 60.1)
- added C2: C, Capacitor_SMD:C_0805_2012Metric_Pad1.18x1.45mm_HandSolder, F.Cu at (147.4, 110.1)
- added C5: C, Capacitor_SMD:C_0805_2012Metric_Pad1.18x1.45mm_HandSolder, F.Cu at (69.0, 129.5)
- added C5: C, Capacitor_SMD:C_0805_2012Metric_Pad1.18x1.45mm_HandSolder, F.Cu at (69.0, 79.5)
- added H1: MountingHole, MountingHole:MountingHole_3.2mm_M3_DIN965, F.Cu at (103.0, 131.0)
- added H1: MountingHole, MountingHole:MountingHole_3.2mm_M3_DIN965, F.Cu at (103.0, 81.0)
- added H2: MountingHole, MountingHole:MountingHole_3.2mm_M3_DIN965, F.Cu at (147.0, 81.0)
- added H2: MountingHole, MountingHole:MountingHole_3.2mm_M3_DIN965, F.Cu at (147.0, 131.0)
- added H3: MountingHole, MountingHole:MountingHole_3.2mm_M3_DIN965, F.Cu at (147.0, 53.0)
- added H3: MountingHole, MountingHole:MountingHole_3.2mm_M3_DIN965, F.Cu at (147.0, 103.0)
- added H4: MountingHole, MountingHole:MountingHole_3.2mm_M3_DIN965, F.Cu at (103.0, 53.0)
- added H4: MountingHole, MountingHole:MountingHole_3.2mm_M3_DIN965, F.Cu at (103.0, 103.0)
- added H5: MountingHole, MountingHole:MountingHole_3.2mm_M3_DIN965, F.Cu at (53.0, 53.0)
- added H5: MountingHole, MountingHole:MountingHole_3.2mm_M3_DIN965, F.Cu at (53.0, 103.0)
- added H6: MountingHole, MountingHole:MountingHole_3.2mm_M3_DIN965, F.Cu at (147.0, 146.0)
- added H6: MountingHole, MountingHole:MountingHole_3.2mm_M3_DIN965, F.Cu at (147.0, 96.0)
- added H7: MountingHole, MountingHole:MountingHole_3.2mm_M3_DIN965, F.Cu at (103.0, 96.0)
- added H7: MountingHole, MountingHole:MountingHole_3.2mm_M3_DIN965, F.Cu at (103.0, 146.0)
- added H8: MountingHole, MountingHole:MountingHole_3.2mm_M3_DIN965, F.Cu at (60.0, 96.0)
- added H8: MountingHole, MountingHole:MountingHole_3.2mm_M3_DIN965, F.Cu at (60.0, 146.0)
- added J1: Conn_01x08_Pin, Connector_JST:JST_EH_B8B-EH-A_1x08_P2.50mm_Vertical, F.Cu at (121.5, 87.6)
- added J1: Conn_01x08_Pin, Connector_JST:JST_EH_B8B-EH-A_1x08_P2.50mm_Vertical, F.Cu at (121.5, 137.6)
- added J10: Conn_01x04_Pin, Connector_JST:JST_EH_B4B-EH-A_1x04_P2.50mm_Vertical, F.Cu at (95.9, 95.1)
- added J10: Conn_01x04_Pin, Connector_JST:JST_EH_B4B-EH-A_1x04_P2.50mm_Vertical, F.Cu at (95.9, 145.1)
- added J11: Conn_01x04_Pin, Connector_JST:JST_EH_B4B-EH-A_1x04_P2.50mm_Vertical, F.Cu at (95.9, 89.3)
- added J11: Conn_01x04_Pin, Connector_JST:JST_EH_B4B-EH-A_1x04_P2.50mm_Vertical, F.Cu at (95.9, 139.3)
- added J12: Conn_01x04_Pin, Connector_JST:JST_EH_B4B-EH-A_1x04_P2.50mm_Vertical, F.Cu at (95.9, 83.5)
- added J12: Conn_01x04_Pin, Connector_JST:JST_EH_B4B-EH-A_1x04_P2.50mm_Vertical, F.Cu at (95.9, 133.5)
- added J13: Conn_01x04_Pin, Connector_JST:JST_EH_B4B-EH-A_1x04_P2.50mm_Vertical, F.Cu at (95.9, 77.7)
- added J13: Conn_01x04_Pin, Connector_JST:JST_EH_B4B-EH-A_1x04_P2.50mm_Vertical, F.Cu at (95.9, 127.7)
- added J14: Conn_01x04_Pin, Connector_JST:JST_EH_B4B-EH-A_1x04_P2.50mm_Vertical, F.Cu at (95.9, 71.8)
- added J14: Conn_01x04_Pin, Connector_JST:JST_EH_B4B-EH-A_1x04_P2.50mm_Vertical, F.Cu at (95.9, 121.8)
- added J15: Conn_01x04_Pin, Connector_JST:JST_EH_B4B-EH-A_1x04_P2.50mm_Vertical, F.Cu at (95.9, 116.0)
- added J15: Conn_01x04_Pin, Connector_JST:JST_EH_B4B-EH-A_1x04_P2.50mm_Vertical, F.Cu at (95.9, 66.0)
- added J16: Conn_01x04_Pin, Connector_JST:JST_EH_B4B-EH-A_1x04_P2.50mm_Vertical, F.Cu at (95.9, 110.2)
- added J16: Conn_01x04_Pin, Connector_JST:JST_EH_B4B-EH-A_1x04_P2.50mm_Vertical, F.Cu at (95.9, 60.2)
- added J17: Conn_01x04_Pin, Connector_JST:JST_EH_B4B-EH-A_1x04_P2.50mm_Vertical, F.Cu at (95.9, 104.4)
- added J17: Conn_01x04_Pin, Connector_JST:JST_EH_B4B-EH-A_1x04_P2.50mm_Vertical, F.Cu at (95.9, 54.4)
- added J18: Conn_01x02_Pin, Connector_JST:JST_EH_S2B-EH_1x02_P2.50mm_Horizontal, F.Cu at (70.2, 83.0)
- added J18: Conn_01x02_Pin, Connector_JST:JST_EH_S2B-EH_1x02_P2.50mm_Horizontal, F.Cu at (70.2, 133.0)
- added J2: Conn_01x08_Pin, Connector_JST:JST_EH_B8B-EH-A_1x08_P2.50mm_Vertical, F.Cu at (146.0, 87.6)
- added J2: Conn_01x08_Pin, Connector_JST:JST_EH_B8B-EH-A_1x08_P2.50mm_Vertical, F.Cu at (146.0, 137.6)
- added J3: Conn_02x06_Odd_Even, Connector_PinHeader_2.54mm:PinHeader_2x06_P2.54mm_Vertical, F.Cu at (121.2, 103.2)
- added J3: Conn_02x06_Odd_Even, Connector_PinHeader_2.54mm:PinHeader_2x06_P2.54mm_Vertical, F.Cu at (121.2, 53.2)
- added J8: Conn_02x10_Odd_Even, Connector_PinHeader_2.54mm:PinHeader_2x10_P2.54mm_Vertical, F.Cu at (82.5, 147.1)
- added J8: Conn_02x10_Odd_Even, Connector_PinHeader_2.54mm:PinHeader_2x10_P2.54mm_Vertical, F.Cu at (82.5, 97.1)
- added J9: Conn_02x10_Odd_Even, Connector_PinHeader_2.54mm:PinHeader_2x10_P2.54mm_Vertical, F.Cu at (54.5, 97.1)
- added J9: Conn_02x10_Odd_Even, Connector_PinHeader_2.54mm:PinHeader_2x10_P2.54mm_Vertical, F.Cu at (54.5, 147.1)
- added R1: R, Resistor_SMD:R_0805_2012Metric_Pad1.20x1.40mm_HandSolder, F.Cu at (108.0, 132.0)
- added R1: R, Resistor_SMD:R_0805_2012Metric_Pad1.20x1.40mm_HandSolder, F.Cu at (108.0, 82.0)
- added R10: R, Resistor_SMD:R_0805_2012Metric_Pad1.20x1.40mm_HandSolder, F.Cu at (128.4, 82.0)
- added R10: R, Resistor_SMD:R_0805_2012Metric_Pad1.20x1.40mm_HandSolder, F.Cu at (128.4, 132.0)
- added R11: R, Resistor_SMD:R_0805_2012Metric_Pad1.20x1.40mm_HandSolder, F.Cu at (130.7, 132.0)
- added R11: R, Resistor_SMD:R_0805_2012Metric_Pad1.20x1.40mm_HandSolder, F.Cu at (130.7, 82.0)
- added R12: R, Resistor_SMD:R_0805_2012Metric_Pad1.20x1.40mm_HandSolder, F.Cu at (132.9, 82.0)
- added R12: R, Resistor_SMD:R_0805_2012Metric_Pad1.20x1.40mm_HandSolder, F.Cu at (132.9, 132.0)
- added R13: R, Resistor_SMD:R_0805_2012Metric_Pad1.20x1.40mm_HandSolder, F.Cu at (135.2, 82.0)
- added R13: R, Resistor_SMD:R_0805_2012Metric_Pad1.20x1.40mm_HandSolder, F.Cu at (135.2, 132.0)
- added R14: R, Resistor_SMD:R_0805_2012Metric_Pad1.20x1.40mm_HandSolder, F.Cu at (137.5, 82.0)
- added R14: R, Resistor_SMD:R_0805_2012Metric_Pad1.20x1.40mm_HandSolder, F.Cu at (137.5, 132.0)
- added R15: R, Resistor_SMD:R_0805_2012Metric_Pad1.20x1.40mm_HandSolder, F.Cu at (139.7, 132.0)
- added R15: R, Resistor_SMD:R_0805_2012Metric_Pad1.20x1.40mm_HandSolder, F.Cu at (139.7, 82.0)
- added R16: R, Resistor_SMD:R_0805_2012Metric_Pad1.20x1.40mm_HandSolder, F.Cu at (142.0, 132.0)
- added R16: R, Resistor_SMD:R_0805_2012Metric_Pad1.20x1.40mm_HandSolder, F.Cu at (142.0, 82.0)
- added R17: R, Resistor_SMD:R_0805_2012Metric_Pad1.20x1.40mm_HandSolder, F.Cu at (103.0, 66.2)
- added R17: R, Resistor_SMD:R_0805_2012Metric_Pad1.20x1.40mm_HandSolder, F.Cu at (103.0, 116.2)
- added R18: R, Resistor_SMD:R_0805_2012Metric_Pad1.20x1.40mm_HandSolder, F.Cu at (105.9, 66.2)
- added R18: R, Resistor_SMD:R_0805_2012Metric_Pad1.20x1.40mm_HandSolder, F.Cu at (105.9, 116.2)
- added R19: R, Resistor_SMD:R_0805_2012Metric_Pad1.20x1.40mm_HandSolder, F.Cu at (108.9, 116.2)
- added R19: R, Resistor_SMD:R_0805_2012Metric_Pad1.20x1.40mm_HandSolder, F.Cu at (108.9, 66.2)
- added R2: R, Resistor_SMD:R_0805_2012Metric_Pad1.20x1.40mm_HandSolder, F.Cu at (110.3, 82.0)
- added R2: R, Resistor_SMD:R_0805_2012Metric_Pad1.20x1.40mm_HandSolder, F.Cu at (110.3, 132.0)
- added R20: R, Resistor_SMD:R_0805_2012Metric_Pad1.20x1.40mm_HandSolder, F.Cu at (111.8, 116.2)
- added R20: R, Resistor_SMD:R_0805_2012Metric_Pad1.20x1.40mm_HandSolder, F.Cu at (111.8, 66.2)
- added R21: R, Resistor_SMD:R_0805_2012Metric_Pad1.20x1.40mm_HandSolder, F.Cu at (114.7, 116.2)
- added R21: R, Resistor_SMD:R_0805_2012Metric_Pad1.20x1.40mm_HandSolder, F.Cu at (114.7, 66.2)
- added R22: R, Resistor_SMD:R_0805_2012Metric_Pad1.20x1.40mm_HandSolder, F.Cu at (117.7, 116.2)
- added R22: R, Resistor_SMD:R_0805_2012Metric_Pad1.20x1.40mm_HandSolder, F.Cu at (117.7, 66.2)
- added R23: R, Resistor_SMD:R_0805_2012Metric_Pad1.20x1.40mm_HandSolder, F.Cu at (120.6, 116.2)
- added R23: R, Resistor_SMD:R_0805_2012Metric_Pad1.20x1.40mm_HandSolder, F.Cu at (120.6, 66.2)
- added R24: R, Resistor_SMD:R_0805_2012Metric_Pad1.20x1.40mm_HandSolder, F.Cu at (123.5, 116.2)
- added R24: R, Resistor_SMD:R_0805_2012Metric_Pad1.20x1.40mm_HandSolder, F.Cu at (123.5, 66.2)
- added R25: R, Resistor_SMD:R_0805_2012Metric_Pad1.20x1.40mm_HandSolder, F.Cu at (126.5, 116.2)
- added R25: R, Resistor_SMD:R_0805_2012Metric_Pad1.20x1.40mm_HandSolder, F.Cu at (126.5, 66.2)
- added R26: R, Resistor_SMD:R_0805_2012Metric_Pad1.20x1.40mm_HandSolder, F.Cu at (129.4, 66.2)
- added R26: R, Resistor_SMD:R_0805_2012Metric_Pad1.20x1.40mm_HandSolder, F.Cu at (129.4, 116.2)
- added R27: R, Resistor_SMD:R_0805_2012Metric_Pad1.20x1.40mm_HandSolder, F.Cu at (132.3, 116.2)
- added R27: R, Resistor_SMD:R_0805_2012Metric_Pad1.20x1.40mm_HandSolder, F.Cu at (132.3, 66.2)
- added R28: R, Resistor_SMD:R_0805_2012Metric_Pad1.20x1.40mm_HandSolder, F.Cu at (135.3, 116.2)
- added R28: R, Resistor_SMD:R_0805_2012Metric_Pad1.20x1.40mm_HandSolder, F.Cu at (135.3, 66.2)
- added R29: R, Resistor_SMD:R_0805_2012Metric_Pad1.20x1.40mm_HandSolder, F.Cu at (138.2, 66.2)
- added R29: R, Resistor_SMD:R_0805_2012Metric_Pad1.20x1.40mm_HandSolder, F.Cu at (138.2, 116.2)
- added R3: R, Resistor_SMD:R_0805_2012Metric_Pad1.20x1.40mm_HandSolder, F.Cu at (112.5, 82.0)
- added R3: R, Resistor_SMD:R_0805_2012Metric_Pad1.20x1.40mm_HandSolder, F.Cu at (112.5, 132.0)
- added R30: R, Resistor_SMD:R_0805_2012Metric_Pad1.20x1.40mm_HandSolder, F.Cu at (141.1, 116.2)
- added R30: R, Resistor_SMD:R_0805_2012Metric_Pad1.20x1.40mm_HandSolder, F.Cu at (141.1, 66.2)
- added R31: R, Resistor_SMD:R_0805_2012Metric_Pad1.20x1.40mm_HandSolder, F.Cu at (144.1, 66.2)
- added R31: R, Resistor_SMD:R_0805_2012Metric_Pad1.20x1.40mm_HandSolder, F.Cu at (144.1, 116.2)
- added R32: R, Resistor_SMD:R_0805_2012Metric_Pad1.20x1.40mm_HandSolder, F.Cu at (147.0, 66.2)
- added R32: R, Resistor_SMD:R_0805_2012Metric_Pad1.20x1.40mm_HandSolder, F.Cu at (147.0, 116.2)
- added R33: R, Resistor_SMD:R_0805_2012Metric_Pad1.20x1.40mm_HandSolder, F.Cu at (119.4, 109.1)
- added R33: R, Resistor_SMD:R_0805_2012Metric_Pad1.20x1.40mm_HandSolder, F.Cu at (119.4, 59.1)
- added R34: R, Resistor_SMD:R_0805_2012Metric_Pad1.20x1.40mm_HandSolder, F.Cu at (58.8, 74.2)
- added R34: R, Resistor_SMD:R_0805_2012Metric_Pad1.20x1.40mm_HandSolder, F.Cu at (58.8, 124.2)
- added R35: R, Resistor_SMD:R_0805_2012Metric_Pad1.20x1.40mm_HandSolder, F.Cu at (58.8, 132.0)
- added R35: R, Resistor_SMD:R_0805_2012Metric_Pad1.20x1.40mm_HandSolder, F.Cu at (58.8, 82.0)
- added R36: R, Resistor_SMD:R_0805_2012Metric_Pad1.20x1.40mm_HandSolder, F.Cu at (58.8, 137.0)
- added R36: R, Resistor_SMD:R_0805_2012Metric_Pad1.20x1.40mm_HandSolder, F.Cu at (58.8, 87.0)
- added R4: R, Resistor_SMD:R_0805_2012Metric_Pad1.20x1.40mm_HandSolder, F.Cu at (114.8, 82.0)
- added R4: R, Resistor_SMD:R_0805_2012Metric_Pad1.20x1.40mm_HandSolder, F.Cu at (114.8, 132.0)
- added R5: R, Resistor_SMD:R_0805_2012Metric_Pad1.20x1.40mm_HandSolder, F.Cu at (117.1, 132.0)
- added R5: R, Resistor_SMD:R_0805_2012Metric_Pad1.20x1.40mm_HandSolder, F.Cu at (117.1, 82.0)
- added R6: R, Resistor_SMD:R_0805_2012Metric_Pad1.20x1.40mm_HandSolder, F.Cu at (119.3, 82.0)
- added R6: R, Resistor_SMD:R_0805_2012Metric_Pad1.20x1.40mm_HandSolder, F.Cu at (119.3, 132.0)
- added R7: R, Resistor_SMD:R_0805_2012Metric_Pad1.20x1.40mm_HandSolder, F.Cu at (121.6, 82.0)
- added R7: R, Resistor_SMD:R_0805_2012Metric_Pad1.20x1.40mm_HandSolder, F.Cu at (121.6, 132.0)
- added R8: R, Resistor_SMD:R_0805_2012Metric_Pad1.20x1.40mm_HandSolder, F.Cu at (123.9, 132.0)
- added R8: R, Resistor_SMD:R_0805_2012Metric_Pad1.20x1.40mm_HandSolder, F.Cu at (123.9, 82.0)
- added R9: R, Resistor_SMD:R_0805_2012Metric_Pad1.20x1.40mm_HandSolder, F.Cu at (126.1, 82.0)
- added R9: R, Resistor_SMD:R_0805_2012Metric_Pad1.20x1.40mm_HandSolder, F.Cu at (126.1, 132.0)
- added U1: TCMT4100, Package_SO:SOP-16_4.4x10.4mm_P1.27mm, F.Cu at (106.9, 73.0)
- added U1: TCMT4100, Package_SO:SOP-16_4.4x10.4mm_P1.27mm, F.Cu at (106.9, 123.0)
- added U2: TCMT4100, Package_SO:SOP-16_4.4x10.4mm_P1.27mm, F.Cu at (118.9, 123.0)
- added U2: TCMT4100, Package_SO:SOP-16_4.4x10.4mm_P1.27mm, F.Cu at (118.9, 73.0)
- added U3: TCMT4100, Package_SO:SOP-16_4.4x10.4mm_P1.27mm, F.Cu at (131.0, 73.0)
- added U3: TCMT4100, Package_SO:SOP-16_4.4x10.4mm_P1.27mm, F.Cu at (131.0, 123.0)
- added U4: TCMT4100, Package_SO:SOP-16_4.4x10.4mm_P1.27mm, F.Cu at (143.0, 73.0)
- added U4: TCMT4100, Package_SO:SOP-16_4.4x10.4mm_P1.27mm, F.Cu at (143.0, 123.0)
- added U5: MCP23017_SS, Package_SO:SSOP-28_5.3x10.2mm_P0.65mm, F.Cu at (137.0, 56.4)
- added U5: MCP23017_SS, Package_SO:SSOP-28_5.3x10.2mm_P0.65mm, F.Cu at (137.0, 106.4)
Routing:
- net +5V: track 0.00 -> 467.7 mm, vias 0 -> 36
- net GND2: track 0.00 -> 325.1 mm, vias 0 -> 34
- net SCK: track 0.00 -> 286.5 mm, vias 0 -> 4
- net SDA: track 0.00 -> 281.1 mm, vias 0 -> 4
- net INT: track 0.00 -> 219.8 mm, vias 0 -> 6
- net GND: track 0.00 -> 87.9 mm, vias 0 -> 76
- net Net-(U5-GPA0): track 0.00 -> 78.8 mm
- net Net-(U5-GPA1): track 0.00 -> 73.2 mm
- net Net-(U5-GPA2): track 0.00 -> 66.5 mm
- net Net-(U5-GPA3): track 0.00 -> 60.5 mm
- net Net-(U5-GPA4): track 0.00 -> 52.8 mm
- net Net-(U5-~{RESET}): track 0.00 -> 48.9 mm, vias 0 -> 4
- net Net-(U5-GPA5): track 0.00 -> 47.0 mm
- net Net-(U5-GPB1): track 0.00 -> 43.1 mm
- net Net-(U5-GPB0): track 0.00 -> 42.2 mm
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- added copper zone on B.Cu, net GND
- added copper zone on F.Cu, net GND
Other:
- board outline added: 100 x 100 mm
- board text added: "24V|GND24"
- board text added: "GND|5V|SDA|SCK"
- board text added: "GND|5V|SDA|SCK|INT|GND24"
- board text added: "INPUT BOARD ONLY V1.1"
- board text added: "OLIMEX ESP32-POE"
